File: Hardware/SparkFun_Qwiic_FS3000.brd (EAGLE design)
At the start: 25.4 x 25.4 mm, 40 parts, among them J2 QWIIC_RA, U1 FS3000

Commit message: Layout done
Parts:
- added U$10: (no value), output:#VCM#0
- added U$13: (no value), output:#ADCR#0
- added U$14: (no value), output:FS30001
- added U$15: (no value), output:#ADC#REF#0
- added U$16, U$20: (no value), output:VELOCITY30003
- added U$18: (no value), output:AIR30004
- added U$19, U$22: (no value), output:SENSOR30005
- added U$3: (no value), output:#SCL#0
- added U$4: (no value), output:#SDA#0
- LOGO2: value SFE_LOGO_NAME_FLAME.1_INCH -> SFE_LOGO_FLAME.1_INCH; device SparkFun-Aesthetics:SFE_LOGO_NAME_FLAME_.1 -> SparkFun-Aesthetics:SFE_LOGO_FLAME_.1
- U$17: device output:FS30000 -> output:FS30001
- U$21: device output:AIR_VELOCITY_SENSOR0 -> output:AIR30004
- moved LOGO1 31.7 mm to (17.3, 10.9), flipped to the bottom, turned to 90 degrees
- moved LOGO3 29.0 mm to (8.26, 18.2)
- moved U$17 26.7 mm to (10.4, 12.6), flipped to the bottom, turned to 90 degrees
- moved U$12 25.6 mm to (8.76, 12.3), turned to 90 degrees
- moved U$21 23.8 mm to (14.6, 12.8), flipped to the bottom, turned to 90 degrees
- moved ADC-REF 4.51 mm to (6.35, 24.0)
- moved LOGO2 4.05 mm to (17.3, 14.4), turned to 90 degrees
- moved R4 2.20 mm to (5.71, 18.8), turned to 180 degrees
- moved U$27 2.05 mm to (1.09, 19.5)
- moved C2 1.91 mm to (14.5, 15.7)
- moved I2C 1.91 mm to (2.84, 17.5)
- moved JP1 1.40 mm to (1.65, 8.00)
- moved U$24 1.40 mm to (1.65, 8.64)
- moved R3 0.90 mm to (5.71, 20.0), turned to 180 degrees
- moved JP11 0.48 mm to (24.5, 8.99)
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Routing:
- net SDA: track 0.00 -> 40.0 mm, vias 0 -> 4
- net SCL: track 0.00 -> 38.0 mm, vias 0 -> 3
- net ADC-REF: track 0.00 -> 17.4 mm
- net VCM: track 1.76 -> 18.5 mm, vias 0 -> 1
- net 3.3V: track 29.0 -> 44.2 mm, vias 1 -> 2
- net N$8: track 0.00 -> 6.99 mm, vias 0 -> 1
- net N$2: track 0.00 -> 5.63 mm, vias 0 -> 1
- net N$1: track 0.00 -> 3.51 mm, vias 0 -> 1
- net N$6: track 0.00 -> 1.78 mm
Other:
- outline, holes or cut-outs redrawn
- board text removed: "FLOW"

Commit message: ran checklist pre-group review
-DRC update
-measures update
-paste reduced on IC pads
Parts:
- moved FRAME1 5.24 mm to (-16.5, -12.7)
- moved LOGO3 4.67 mm to (7.09, 22.7)
Other:
- board text added: "Measure Units: INCHES"
