File: Hardware/Option_2/SparkFun_Qwiic_FS3000_top.brd (EAGLE design)
At the start: 25.4 x 25.4 mm, 56 parts, among them J2 QWIIC_RA, J3 QWIIC_RA, U1 FS3000

Commit message: Group Review Changes
-Buzzard labels on VCM/ADCR changed to be correct inputs/outputs end type
-Added in solder pads for two versions (7.23m/s vs 15m/s) (1005/1015)
-Moved"supply range" to below the IC and change to "VDD range".
-schematic cleanup - power LED jumper paragraph. space in I2C address.
-added space between "I2C address" and "0x28" in board silk
-added name/flame logo to board silk.
Parts:
- removed LOGO2: SFE_LOGO_FLAME.1_INCH, SparkFun-Aesthetics:SFE_LOGO_FLAME_.1
- added LOGO5: SFE_LOGO_NAME_FLAME.1_INCH, SparkFun-Aesthetics:SFE_LOGO_NAME_FLAME_.1
- added U$28: (no value), output:I2C_ADD#_0X280
- added U$29: (no value), output:10150
- LOGO3: value SFE_LOGO_FLAME.1_INCH -> SFE_LOGO_NAME_FLAME.1_INCH; device SparkFun-Aesthetics:SFE_LOGO_FLAME_.1 -> SparkFun-Aesthetics:SFE_LOGO_NAME_FLAME_.1
- U$12: device output:I2C_ADD#0X280 -> output:10050
- moved LOGO1 20.5 mm to (2.51, 19.2)
- moved U$12 15.3 mm to (23.4, 19.4), flipped to the top
- moved LOGO3 13.0 mm to (12.7, 10.2), flipped to the bottom
- moved U$17 8.36 mm to (19.1, 15.2)
- moved U$20 8.36 mm to (18.9, 18.1)
- moved U$21 8.36 mm to (18.8, 19.5)
- moved U$22 8.36 mm to (19.1, 16.8)
- moved U$18 4.70 mm to (9.27, 10.3)
- moved U$16 2.98 mm to (14.1, 10.3)
- moved U$14 2.44 mm to (12.6, 7.37)
- moved U$19 2.32 mm to (12.6, 8.89)
Changed lines of the file:
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@@
 <layer number="27" name="tValues" color="7" fill="1" visible="no" active="yes"/>
 <layer number="28" name="bValues" color="7" fill="1" visible="no" active="yes"/>
-<layer number="29" name="tStop" color="7" fill="3" visible="no" active="yes"/>
+<layer number="29" name="tStop" color="7" fill="3" visible="yes" active="yes"/>
 <layer number="30" name="bStop" color="7" fill="6" visible="no" active="yes"/>
-<layer number="31" name="tCream" color="7" fill="4" visible="no" active="yes"/>
+<layer number="31" name="tCream" color="7" fill="4" visible="yes" active="yes"/>
 <layer number="32" name="bCream" color="7" fill="5" visible="no" active="yes"/>
 <layer number="33" name="tFinish" color="6" fill="3" visible="no" active="yes"/>
@@
 <layer number="47" name="Measures" color="7" fill="1" visible="no" active="yes"/>
 <layer number="48" name="Document" color="7" fill="1" visible="no" active="yes"/>
-<layer number="49" name="Reference" color="7" fill="1" visible="no" active="yes"/>
+<layer number="49" name="Reference" color="7" fill="1" visible="yes" active="yes"/>
 <layer number="50" name="dxf" color="7" fill="1" visible="no" active="yes"/>
 <layer number="51" name="tDocu" color="6" fill="1" visible="yes" active="yes"/>
@@
 <wire x1="12.065" y1="15.4178" x2="12.6746" y2="15.0368" width="0.1524" layer="22"/>
 <wire x1="12.6746" y1="15.0368" x2="13.3096" y2="15.4686" width="0.1524" layer="22"/>
+<rectangle x1="20.3454" y1="18.7706" x2="21.8694" y2="20.2184" layer="31"/>
+<rectangle x1="20.5359" y1="18.9484" x2="20.9804" y2="20.0279" layer="29"/>
+<rectangle x1="21.1709" y1="18.9484" x2="21.6154" y2="20.0279" layer="29"/>
+<rectangle x1="20.5105" y1="17.272" x2="20.955" y2="18.3515" layer="29"/>
+<rectangle x1="21.1455" y1="17.272" x2="21.59" y2="18.3515" layer="29"/>
 </plain>
 <attributes>
@@
 <attribute name="VALUE" x="6.7056" y="21.59" size="0.6096" layer="27" font="vector" ratio="20" rot="R270" align="top-center"/>
 </element>
-<element name="LOGO1" library="SparkFun-Aesthetics" package="OSHW-LOGO-MINI" value="OSHW-LOGOMINI" x="22.0726" y="13.081" smashed="yes" rot="MR0"/>
+<element name="LOGO1" library="SparkFun-Aesthetics" package="OSHW-LOGO-MINI" value="OSHW-LOGOMINI" x="2.5146" y="19.177" smashed="yes" rot="MR0"/>
 <element name="JP11" library="SparkFun" package="MICRO-FIDUCIAL" value="FIDUCIALUFIDUCIAL" x="24.638" y="0.7366" smashed="yes" rot="MR0"/>
 <element name="JP5" library="SparkFun" package="MICRO-FIDUCIAL" value="FIDUCIALUFIDUCIAL" x="0.762" y="24.638" smashed="yes" rot="MR0"/>
@@
 <element name="U$24" library="output" package="#LED#0" value="" x="1.651" y="8.636" smashed="yes" rot="MR90"/>
 <element name="U$25" library="output" package="PWR0" value="" x="2.6416" y="7.8486" smashed="yes"/>
-<element name="LOGO3" library="SparkFun-Aesthetics" package="SFE_LOGO_FLAME_.1" value="SFE_LOGO_FLAME.1_INCH" x="22.5298" y="18.6436" smashed="yes"/>
 <element name="U$27" library="output" package="#I2C#0" value="" x="22.2758" y="8.382" smashed="yes" rot="MR90"/>
 <element name="C2" library="SparkFun-Capacitors" package="0402-TIGHT" value="0.1uF" x="7.4676" y="23.876" smashed="yes" rot="R90">
@@
 <attribute name="VALUE" x="18.415" y="23.876" size="0.6096" layer="27" font="vector" ratio="20" rot="R90" align="top-center"/>
 </element>
-<element name="U$12" library="output" package="I2C_ADD#0X280" value="" x="13.1826" y="7.9756" smashed="yes" rot="MR0"/>
 <element name="U1" library="FS3000" package="FS3000" value="FS3000" x="12.7" y="20.828" smashed="yes">
 <attribute name="NAME" x="10.9855" y="25.48255" size="0.6096" layer="25" font="vector" ratio="20"/>
@@
 <element name="U$10" library="output" package="#VCM#0" value="" x="16.51" y="1.651" smashed="yes" rot="MR90"/>
 <element name="U$13" library="output" package="#ADCR#0" value="" x="19.05" y="1.524" smashed="yes" rot="MR90"/>
-<element name="U$14" library="output" package="FS30001" value="" x="12.192" y="9.779" smashed="yes"/>
-<element name="U$16" library="output" package="VELOCITY30003" value="" x="12.192" y="12.573" smashed="yes"/>
-<element name="U$18" library="output" package="AIR30004" value="" x="12.192" y="13.97" smashed="yes"/>
-<element name="U$19" library="output" package="SENSOR30005" value="" x="12.192" y="11.176" smashed="yes"/>
+<element name="U$14" library="output" package="FS30001" value="" x="12.573" y="7.366" smashed="yes"/>
+<element name="U$16" library="output" package="VELOCITY30003" value="" x="14.097" y="10.287" smashed="yes"/>
+<element name="U$18" library="output" package="AIR30004" value="" x="9.271" y="10.287" smashed="yes"/>
+<element name="U$19" library="output" package="SENSOR30005" value="" x="12.573" y="8.89" smashed="yes"/>
 <element name="U$15" library="output" package="#ADC#REF#0" value="" x="6.35" y="23.241" smashed="yes" rot="MR90"/>
-<element name="U$17" library="output" package="FS30001" value="" x="12.954" y="9.525" smashed="yes" rot="MR0"/>
-<element name="U$20" library="output" package="VELOCITY30003" value="" x="12.8016" y="12.4206" smashed="yes" rot="MR0"/>
-<element name="U$21" library="output" package="AIR30004" value="" x="12.6746" y="13.8176" smashed="yes" rot="MR0"/>
-<element name="U$22" library="output" package="SENSOR30005" value="" x="12.954" y="11.0744" smashed="yes" rot="MR0"/>
-<element name="LOGO2" library="SparkFun-Aesthetics" package="SFE_LOGO_FLAME_.1" value="SFE_LOGO_FLAME.1_INCH" x="21.8948" y="17.2466" smashed="yes" rot="MR0"/>
+<element name="U$17" library="output" package="FS30001" value="" x="19.05" y="15.24" smashed="yes" rot="MR0"/>
+<element name="U$20" library="output" package="VELOCITY30003" value="" x="18.8976" y="18.1356" smashed="yes" rot="MR0"/>
+<element name="U$21" library="output" package="AIR30004" value="" x="18.7706" y="19.5326" smashed="yes" rot="MR0"/>
+<element name="U$22" library="output" package="SENSOR30005" value="" x="19.05" y="16.7894" smashed="yes" rot="MR0"/>
 <element name="JP4" library="SparkFun" package="STAND-OFF" value="STAND-OFF" x="22.86" y="22.86" smashed="yes"/>
 <element name="JP7" library="SparkFun" package="STAND-OFF" value="STAND-OFF" x="22.86" y="2.54" smashed="yes"/>
@@
 <element name="U$23" library="output" package="#AIRFLOW#0" value="" x="19.0754" y="19.9644" smashed="yes" rot="R90"/>
 <element name="U$26" library="output" package="#AIRFLOW#0" value="" x="12.6746" y="19.9136" smashed="yes" rot="MR90"/>
+<element name="U$28" library="output" package="I2C_ADD#_0X280" value="" x="19.177" y="13.716" smashed="yes" rot="MR0"/>
+<element name="LOGO5" library="SparkFun-Aesthetics" package="SFE_LOGO_NAME_FLAME_.1" value="SFE_LOGO_NAME_FLAME.1_INCH" x="12.7" y="12.573" smashed="yes"/>
+<element name="U$12" library="output" package="10050" value="" x="23.368" y="19.431" smashed="yes"/>
+<element name="U$29" library="output" package="10150" value="" x="23.241" y="17.78" smashed="yes"/>
+<element name="LOGO3" library="SparkFun-Aesthetics" package="SFE_LOGO_NAME_FLAME_.1" value="SFE_LOGO_NAME_FLAME.1_INCH" x="12.7" y="10.16" smashed="yes" rot="MR0"/>
 </elements>
 <signals>
@@
 <via x="3.6576" y="14.2494" extent="1-16" drill="0.381"/>
 <via x="14.5034" y="8.6614" extent="1-16" drill="0.381"/>
-<via x="12.4968" y="11.7856" extent="1-16" drill="0.381"/>
+<via x="13.5128" y="11.6586" extent="1-16" drill="0.381"/>
 </signal>
 <signal name="SCL">
